File: feathertooth.kicad_pcb (KiCad board)
At the start: 2 copper layers, 50.8 x 22.9 mm, 23 parts, among them J1 TopRow, J2 BottomRow, J3 BAT, J4 USB_B_Micro, J5 Conn_ARM_JTAG_SWD_10, SW1 E_SWITCH, U1 BGM113, U2 MCP1703A, U3 MCP73831-2-OT

Commit message: unfinished USB-C second revision
Parts:
- added R4: 100k, Resistors_SMD:R_0603, F.Cu at (141.0, 82.0)
- J4: value USB_B_Micro -> GT_USB_C; footprint Daniel:SUNTECH_ST-USB-001G -> Daniel:USB_C_Receptacle_GT-USB-7010
- moved R1 26.7 mm to (154.3, 135.3)
- moved U3 26.7 mm to (157.5, 134.6)
- moved C1 26.7 mm to (158.1, 137.8)
- moved C3 26.7 mm to (154.3, 131.4)
- moved R2 26.7 mm to (154.9, 137.8)
- moved SW1 20.2 mm to (171.4, 129.5)
- moved MH3 17.6 mm to (133.3, 123.2)
- moved MH4 17.6 mm to (133.3, 113.0)
- moved D1 16.8 mm to (146.1, 130.8)
- moved R3 9.71 mm to (156.2, 91.4)
- moved D2 9.53 mm to (151.1, 94.0)
- moved J4 0.63 mm to (151.1, 109.2)
Connections:
- C1 pad 1: /Vbat -> Net-(C1-Pad1)
- J1 pad 10: /pb13 -> /swdio
- J1 pad 6: Net-(J1-Pad6) -> /pb11
- J1 pad 7: Net-(J1-Pad7) -> /pb12
- J1 pad 8: /pb11 -> /pb13
- J1 pad 9: /pb12 -> /swdclk
- U1 pad 33: /pd13 -> Net-(U1-Pad33)
- U2 pad 2: /Vbat -> Net-(C1-Pad1)
Routing:
- net /pb11: track 36.8 -> 13.2 mm
- net +3V3: track 74.3 -> 61.1 mm
- net /Vusb: track 31.3 -> 18.3 mm
- net /rst: track 47.0 -> 34.4 mm, vias 3 -> 2
- net GND: track 85.3 -> 75.1 mm
- net /swdclk: track 20.5 -> 26.8 mm, vias 0 -> 1
- net Net-(D1-Pad1): track 4.97 -> 0.00 mm
- net /pb12: track 7.81 -> 11.8 mm
- net /swdio: track 21.0 -> 25.0 mm
- net /pb13: track 7.10 -> 10.3 mm
- net Net-(D2-Pad1): track 3.12 -> 0.00 mm
Other:
- net class PWR added: clearance 0.2, trace_width 0.5, via_dia 0.8, via_drill 0.4
- board text added: "bgm113 feather rev1"
- board text removed: "bgm113 feather rev0"
