File: feathertooth.sch (KiCad schematic (older format))
At the start: 23 parts, among them J1 TopRow, J2 BottomRow, J3 BAT, J4 USB_B_Micro, J5 Conn_ARM_JTAG_SWD_10, SW1 E_SWITCH, U1 BGM113, U2 MCP1703A, U3 MCP73831-2-OT

Commit message: unfinished USB-C second revision
Parts:
- removed J4: USB_B_Micro, Daniel:SUNTECH_ST-USB-001G, symbol Connector:USB_B_Micro
- added D3: D_Schottky, symbol Device:D_Schottky
- added J4: GT_USB_C, Daniel:USB_C_Receptacle_GT-USB-7010, symbol daniel:GT_USB_C
- added Q1: ? P-CH MOSFET, Package_TO_SOT_SMD:SOT-23, symbol Transistor_FET:BSS84
- added R4: 100k, Resistors_SMD:R_0603, symbol Device:R
Connections:
- wire segments 116 -> 134
- no-connect marks 5 -> 9
Other:
- note added: "MCP AN1149"
- moved on the sheet: U3
